File: Main_MOSFET_Cooler.kicad_pcb (KiCad board)
At the start: 2 copper layers, 100 x 100 mm, 18 parts, among them J1 Gate, J2 MOS+, J3 MOS-, J4 Thermister, P1 Eoshi-chan_Silk, P2 Serial_QR, Q1 TK100E06N1, Q2 TK100E06N1

Commit message: before mirror
Parts:
- J2, J3: footprint Akizuki_ScrewTerminal:ScrewTerminal_01x01_PCB-20 -> AM_Conn_ScrewTerminal:ScrewTerminal_01x01_PCB-20
Routing:
- net /NTC-: track 88.0 -> 87.5 mm, vias 2 -> 0
- net /NTC+: track 90.2 -> 89.8 mm, vias 2 -> 0
- net /Gate: vias 0 -> 1
Other:
- board text added: "ELECTRONIC LOAD CPU Cooler Board (v0.1-alpha.2) Designed by: EosinY"
- board text removed: "ELECTRONIC LOAD CPU Cooler Board (v0.1-alpha.1) Designed by: EosinY"
